Commit message: Visualize 2d path in pybullet

File: scripts/darias_energy_control/tiago_single_with_holoBaseCXY.urdf (robot description, URDF)
Before this commit: robot tiago, 50 links, 49 joints
Joints:
- joint X: limit lower=-5.0 upper=5.0 effort=100.0 velocity=0.2 -> lower=-10.0 upper=10.0 effort=100.0 velocity=0.1
- joint Y: limit lower=-5.0 upper=5.0 effort=100.0 velocity=0.2 -> lower=-10.0 upper=10.0 effort=100.0 velocity=0.1
