Commit message: Finish holonomic base+arm OSC

File: robots/tiago/tiago_single_with_holoBaseCXY.urdf (robot description, URDF)
Before this commit: robot tiago, 47 links, 46 joints
Links:
- added link $world1
- added link $world2
- added link world
Joints:
- added joint R: type revolute, parent $world2, child base_footprint, origin xyz=0 0 0 rpy=0 0 0, axis 0 0 1, limit lower=-10.0 upper=10.0 effort=100.0 velocity=1.
- added joint X: type prismatic, parent $world1, child $world2, origin xyz=0 0 0 rpy=0 0 0, axis 1 0 0, limit lower=-10.0 upper=10.0 effort=100.0 velocity=0.1
- added joint Y: type prismatic, parent world, child $world1, origin xyz=0 0 0 rpy=0 0 0, axis 0 1 0, limit lower=-10.0 upper=10.0 effort=100.0 velocity=0.1
- joint ignore_suspension_left_joint: origin xyz=0 0 -0.02 rpy=0 0 0 -> xyz=0 0 0 rpy=0 0 0
- joint ignore_suspension_right_joint: origin xyz=0 0 -0.02 rpy=0 0 0 -> xyz=0 0 0 rpy=0 0 0
- joint wheel_left_joint: axis 0 0 1  -> 0 0 1; type revolute -> fixed
- joint wheel_right_joint: type revolute -> fixed

Commit message: Finish holonomicBase(YXC)+Arm OSC

File: robots/tiago/tiago_single_with_holoBaseCXY.urdf (robot description, URDF)
Before this commit: robot tiago, 50 links, 49 joints
Joints:
- joint R: limit lower=-10.0 upper=10.0 effort=100.0 velocity=1. -> lower=-3.1416 upper=3.1416 effort=100.0 velocity=0.2; type revolute -> continuous

Commit message: Add base_line algorithm and visualize the generated path

File: robots/tiago/tiago_single_with_holoBaseCXY.urdf (robot description, URDF)
Before this commit: robot tiago, 50 links, 49 joints
Joints:
- joint X: child $world2 -> $world1; parent $world1 -> world
- joint Y: child $world1 -> $world2; parent world -> $world1

Commit message: Add _test_simple_tiago_lefthand_base.py

File: robots/tiago/tiago_single_with_holoBaseCXY.urdf (robot description, URDF)
Before this commit: robot tiago, 50 links, 49 joints
Joints:
- joint R: type continuous -> revolute

Commit message: 08.09

File: robots/tiago/tiago_single_with_holoBaseCXY.urdf (robot description, URDF)
Before this commit: robot tiago, 50 links, 49 joints
Joints:
- joint R: type revolute -> continuous
